File: Main Board.sch (EAGLE design)
At the start: 25 parts, among them IC1 TB6612FNG, U1 TPS61030RSAR

Commit message: Whatever man
Parts:
- removed X1: (no value), Adafruit:ANTENNA_U.FL
- added R10, R11, R4, R5, R6, R7, R8, R9: 1.65K Ohms, Vishay:CRCW06031K65FKEA
- added U$20, U$21: MOTOR, GoatFinder:MOTOR
- added U$22, U$23, U$24, U$25, U$26, U$28, U$29, U$30: PJUMP, GoatFinder:PJUMP
- added U$27: PWM, GoatFinder:PWM
- U$15, U$16, U$17: value MOTOR2 -> PJUMP; device GoatFinder:MOTOR2 -> GoatFinder:PJUMP
- U$5: value GPS -> MOTOR; device GoatFinder:GPS -> GoatFinder:MOTOR
Connections:
- removed net GPIO4: U$11.GPIO4, U$5.3D
- removed net GPIO5: U$11.GPIO5, U$5.RESET
- removed net N$13: U$11.SDA0, U$6.SDA
- removed net N$14: U$11.SCL0, U$6.SCL
- removed net N$4: U$11.TXD, U$5.RX
- removed net PWMA: U$11.GPIO23
- removed net PWMB: U$11.GPIO26
- new net HALL1: R5.2, R6.2, U$11.GPIO4
- new net HALL2: R4.2, R7.2, U$11.GPIO5
- new net N$5: R5.1, U$15.VCC
- new net N$6: R4.1, U$16.VCC
- new net PWM0: U$27.PWM2, U$30.VCC
- new net PWM1: U$27.PWM3, U$29.VCC
- new net PWM10: U$26.VCC, U$27.PWM10
- new net PWM2: U$27.PWM4, U$28.VCC
- new net PWM5: U$17.VCC, U$27.PWM5
- new net PWM6: U$22.VCC, U$27.PWM6
- new net PWM7: U$23.VCC, U$27.PWM7
- new net PWM8: U$24.VCC, U$27.PWM8
- new net PWM9: U$25.VCC, U$27.PWM9
- net +3.3V: now also R11.1, R9.1, U$27.A0, U$27.A1, U$27.A2, U$27.VIN; no longer U$5.VCC
- net +5V: now also R10.1, R8.1, U$15.SIG, U$16.SIG
- net GND: now also R6.1, R7.1, U$15.GND, U$16.GND, U$17.GND, U$21.P$2, U$22.GND, U$23.GND, U$24.GND, U$25.GND, U$26.GND, U$27.A3, U$27.A4, U$27.A5, U$27.GND, U$27._OE, U$28.GND, U$29.GND, U$30.GND; no longer U$17.P$2, U$5.GND@1, U$5.GND@2, U$5.GND@3, U$5.GND@4, X1.GND@0, X1.GND@1
- net GPIO0: no longer U$5.1PPS
- net MOTA: now also U$27.PWM0
- net MOTB: now also U$27.PWM1
- net N$10: now also U$27.SCL, U$6.SCL
- net N$12: now also U$27.SDA, U$6.SDA
- net N$16: now also U$20.P$1; no longer U$15.P$1
- net N$17: now also U$20.P$2; no longer U$15.P$2
- net N$18: now also U$5.P$1; no longer U$16.P$1
- net N$19: now also U$5.P$2; no longer U$16.P$2
- net N$3: now also R8.2, R9.2, U$17.SIG, U$22.SIG, U$23.SIG, U$24.SIG, U$25.SIG, U$26.SIG; no longer U$11.RXD, U$5.TX
- net N$8: now also R10.2, R11.2, U$28.SIG, U$29.SIG, U$30.SIG; no longer U$5.ANT, X1.SIGNAL
- net VBAT: now also U$21.P$1; no longer U$17.P$1
